Commit message: ros2_control now move thruster fans but boat still does not move

File: vrx_urdf/tuna_gazebo/urdf/boat_gazebo.urdf (robot description, URDF)
Before this commit: robot tuna, 3 links, 2 joints
Joints:
- joint base_to_prop_left: axis 0 1 0 -> 1 0 0
- joint base_to_prop_right: axis 0 1 0 -> 1 0 0

File: vrx_urdf/wamv_gazebo/urdf/thruster_layouts/wamv_gazebo_thruster_config.xacro (robot description, xacro)
@@ -6,7 +6,5 @@
     <xacro:property name="x_u" value="51.3" />
     <xacro:property name="max_velocity_mps" value="7.71667" />
-    <plugin
-      filename="gz-sim-thruster-system"
-      name="gz::sim::systems::Thruster">
+    <plugin filename="gz-sim-thruster-system" name="gz::sim::systems::Thruster">
       <joint_name>${namespace}/${name}_engine_propeller_joint</joint_name>
       <thrust_coefficient>0.004422</thrust_coefficient>
